Commit message: add

File: xe_lidar/description/gazebo_control_ackermann.xacro (robot description, xacro)
@@ -9,7 +9,10 @@
             <rear_left_joint>rear_left_wheel_joint</rear_left_joint>
             <rear_right_joint>rear_right_wheel_joint</rear_right_joint>
-            <!-- Steering joints - plugin có thể yêu cầu tên đơn giản hơn -->
+            <!-- Steering joints -->
             <left_steering_joint>front_left_steering_joint</left_steering_joint>
             <right_steering_joint>front_right_steering_joint</right_steering_joint>
+            <steering_wheel_joint>steering_wheel_joint</steering_wheel_joint>
+            <!-- Command topic -->
+            <command_topic>cmd_vel</command_topic>
             <!-- Geometry -->
             <wheel_separation>0.28</wheel_separation>

File: xe_lidar/description/lidar.xacro (robot description, xacro)
@@ -34,5 +34,5 @@
             <pose> 0 0 0 0 0 0 </pose>
             <visualize>false</visualize>
-            <update_rate>10</update_rate>
+            <update_rate>20</update_rate>
             <ray>
                 <scan>

File: xe_lidar/description/robot_core_ackermann.xacro (robot description, xacro)
@@ -78,4 +78,33 @@
         <material>Gazebo/Orange</material>
     </gazebo>
+    <!-- STEERING WHEEL JOINT (vô lăng - optional cho plugin) -->
+    <joint name="steering_wheel_joint" type="revolute">
+        <parent link="chassis"/>
+        <child link="steering_wheel_link"/>
+        <origin xyz="0.1 0 0.05" rpy="0 0 0"/>
+        <axis xyz="0 0 1"/>
+        <limit lower="${-max_steer_angle}" upper="${max_steer_angle}" effort="1000" velocity="10"/>
+    </joint>
+    <link name="steering_wheel_link">
+        <visual>
+            <origin xyz="0 0 0" rpy="0 0 0"/>
+            <geometry>
+                <cylinder radius="0.05" length="0.01"/>
+            </geometry>
+            <material name="black"/>
+        </visual>
+        <collision>
+            <origin xyz="0 0 0" rpy="0 0 0"/>
+            <geometry>
+                <cylinder radius="0.05" length="0.01"/>
+            </geometry>
+        </collision>
+        <xacro:inertial_cylinder mass="0.01" length="0.01" radius="0.05">
+            <origin xyz="0 0 0" rpy="0 0 0"/>
+        </xacro:inertial_cylinder>
+    </link>
+    <gazebo reference="steering_wheel_link">
+        <material>Gazebo/Black</material>
+    </gazebo>
     <!-- FRONT LEFT STEERING JOINT -->
     <joint name="front_left_steering_joint" type="revolute">
