Commit message: add

File: xe_lidar/description/robot_core_ackermann.xacro (robot description, xacro)
@@ -2,4 +2,6 @@
 <robot xmlns:xacro="http://www.ros.org/wiki/xacro" >
     <xacro:include filename="inertial_macros.xacro"/>
+    <!-- Math constants -->
+    <xacro:property name="pi" value="3.1415926535897931"/>
     <!-- Properties -->
     <xacro:property name="chassis_length" value="0.49"/>
@@ -14,9 +16,9 @@
     <xacro:property name="front_wheel_x" value="0.2"/>
     <xacro:property name="front_wheel_y" value="0.14"/>
-    <xacro:property name="front_wheel_z" value="0.0"/>
+    <xacro:property name="front_wheel_z" value="${-wheel_radius}"/>  <!-- Bánh xe chạm đất -->
     <!-- Rear wheels (fixed) -->
     <xacro:property name="rear_wheel_x" value="-0.2"/>
     <xacro:property name="rear_wheel_y" value="0.14"/>
-    <xacro:property name="rear_wheel_z" value="0.0"/>
+    <xacro:property name="rear_wheel_z" value="${-wheel_radius}"/>  <!-- Bánh xe chạm đất -->
     <!-- Wheelbase (khoảng cách giữa bánh trước và sau) -->
     <xacro:property name="wheelbase" value="0.4"/>
