Commit message: add

File: xe_lidar/description/robot_ackermann.urdf.xacro (robot description, xacro)
@@ -3,4 +3,6 @@
     <xacro:arg name="use_ros2_control" default="true"/>
     <xacro:arg name="sim_mode" default="false"/>
+    <!-- Math constants - define before including other files -->
+    <xacro:property name="pi" value="3.1415926535897931"/>
     <xacro:include filename="robot_core_ackermann.xacro" />
     <xacro:if value="$(arg use_ros2_control)">

File: xe_lidar/description/robot_core_ackermann.xacro (robot description, xacro)
@@ -2,6 +2,4 @@
 <robot xmlns:xacro="http://www.ros.org/wiki/xacro" >
     <xacro:include filename="inertial_macros.xacro"/>
-    <!-- Math constants -->
-    <xacro:property name="pi" value="3.1415926535897931"/>
     <!-- Properties -->
     <xacro:property name="chassis_length" value="0.49"/>

Commit message: add

File: xe_lidar/description/robot_ackermann.urdf.xacro (robot description, xacro)
@@ -3,6 +3,6 @@
     <xacro:arg name="use_ros2_control" default="true"/>
     <xacro:arg name="sim_mode" default="false"/>
-    <!-- Math constants - define before including other files -->
-    <xacro:property name="pi" value="3.1415926535897931"/>
+    <!-- Include constants first -->
+    <xacro:include filename="constants.xacro" />
     <xacro:include filename="robot_core_ackermann.xacro" />
     <xacro:if value="$(arg use_ros2_control)">
