Commit message: add

File: xe_lidar/description/camera.xacro (robot description, xacro)
@@ -4,5 +4,6 @@
         <parent link="chassis"/>
         <child link="camera_link"/>
-        <origin xyz="0.276 0 0.181" rpy="0 0.18 0"/>
+        <!-- Camera quay xuống nhìn đường (pitch -0.7 radian ≈ -40 độ) -->
+        <origin xyz="0.276 0 0.181" rpy="0 -0.7 0"/>
     </joint>
     <link name="camera_link">

Commit message: add

File: xe_lidar/description/camera.xacro (robot description, xacro)
@@ -4,6 +4,6 @@
         <parent link="chassis"/>
         <child link="camera_link"/>
-        <!-- Camera quay xuống nhìn đường (pitch -0.7 radian ≈ -40 độ) -->
-        <origin xyz="0.276 0 0.181" rpy="0 -0.7 0"/>
+        <!-- Camera đặt trên cao và nhìn thẳng xuống (pitch -1.4 radian ≈ -80 độ) -->
+        <origin xyz="0.0 0 0.6" rpy="0 -1.4 0"/>
     </joint>
     <link name="camera_link">

Commit message: add

File: xe_lidar/description/camera.xacro (robot description, xacro)
@@ -4,6 +4,6 @@
         <parent link="chassis"/>
         <child link="camera_link"/>
-        <!-- Camera đặt trên cao và nhìn thẳng xuống (pitch -1.4 radian ≈ -80 độ) -->
-        <origin xyz="0.0 0 0.6" rpy="0 -1.4 0"/>
+        <!-- Camera đặt trên cao và nhìn thẳng xuống (pitch 1.4 radian ≈ 80 độ để đảo ngược hướng) -->
+        <origin xyz="0.0 0 1.2" rpy="0 1.4 0"/>
     </joint>
     <link name="camera_link">

Commit message: Fix critical Ackermann steering control bugs and update documentation
Major fixes:
1. Fix angular.z control logic (removed incorrect negative sign)
   - Before: offset > 0 → turn right (WRONG, makes car drift more!)
   - After: offset > 0 → turn left (CORRECT, brings car back to center)

2. Fix slope classification for lane detection
   - Before: left lane = negative slope (WRONG in image coordinates)
   - After: left lane = positive slope (CORRECT, Y increases downward)

3. Fix camera pitch angle (1.4 rad → 0.4 rad)
   - Before: 80° too steep, only sees very close to car
   - After: 23° appropriate angle for road ahead

4. Add angular velocity limits for Ackermann steering
   - Respect max_steer_angle constraint (~30°)
   - Prevent excessive steering commands

5. Fix comments and priority logic
   - Clarify LiDAR has higher priority than Camera
   - Update all misleading comments

6. Rewrite comprehensive README
   - Explain all bugs fixed
   - Detailed Ackermann steering theory
   - Complete installation and usage guide
   - Troubleshooting section

Files changed:
- xe_lidar/scripts/obstacle_avoidance.py: Core control logic fixes
- xe_lidar/description/camera.xacro: Camera angle adjustment
- readme.md: Complete rewrite with detailed documentation

File: xe_lidar/description/camera.xacro (robot description, xacro)
@@ -4,6 +4,9 @@
         <parent link="chassis"/>
         <child link="camera_link"/>
-        <!-- Camera đặt trên cao và nhìn thẳng xuống (pitch 1.4 radian ≈ 80 độ để đảo ngược hướng) -->
-        <origin xyz="0.0 0 1.2" rpy="0 1.4 0"/>
+        <!-- Camera đặt trên cao và nghiêng xuống để nhìn đường
+             Position: x=0.2m (phía trước), y=0 (giữa), z=0.25m (cao 25cm từ chassis)
+             Orientation: pitch=0.4 radian (≈ 23°) để nhìn xuống đường phía trước
+             (Không dùng 1.4 rad vì quá dốc, sẽ chỉ nhìn thấy gần xe) -->
+        <origin xyz="0.2 0 0.25" rpy="0 0.4 0"/>
     </joint>
     <link name="camera_link">

Commit message: Revert camera angle - overhead camera setup is correct
Camera setup clarification:
- The camera in simulation is an OVERHEAD camera (bird's eye view)
- Position: z=1.2m above chassis
- Pitch: 1.4 rad (≈80°) looking down
- This is correct for simulation lane detection from top-down view
- NOT a forward-facing camera like on real cars

Previous commit incorrectly changed this to forward-facing camera.
Original setup is the intended design for simulation.

Updated README:
- Removed camera angle from bug list (it was not a bug)
- Now only lists 4 critical bugs that were fixed:
  1. Angular.z control logic (inverted sign)
  2. Slope classification (left/right lane detection)
  3. Missing angular velocity limits for Ackermann
  4. Misleading comments and priority logic

Files changed:
- xe_lidar/description/camera.xacro: Reverted to original overhead setup
- readme.md: Updated to reflect only actual bugs (removed camera angle)

File: xe_lidar/description/camera.xacro (robot description, xacro)
@@ -4,9 +4,9 @@
         <parent link="chassis"/>
         <child link="camera_link"/>
-        <!-- Camera đặt trên cao và nghiêng xuống để nhìn đường
-             Position: x=0.2m (phía trước), y=0 (giữa), z=0.25m (cao 25cm từ chassis)
-             Orientation: pitch=0.4 radian (≈ 23°) để nhìn xuống đường phía trước
-             (Không dùng 1.4 rad vì quá dốc, sẽ chỉ nhìn thấy gần xe) -->
-        <origin xyz="0.2 0 0.25" rpy="0 0.4 0"/>
+        <!-- Camera đặt trên cao và nhìn xuống (bird's eye view / overhead camera)
+             Position: x=0, y=0, z=1.2m (cao 1.2m phía trên chassis)
+             Orientation: pitch=1.4 rad (≈ 80°) để nhìn gần như thẳng xuống
+             Setup này cho phép camera nhìn vạch kẻ đường từ góc trên cao (simulation) -->
+        <origin xyz="0.0 0 1.2" rpy="0 1.4 0"/>
     </joint>
     <link name="camera_link">

Commit message: Fix camera pitch: change from positive to negative (look down instead of up)
Critical fix for camera orientation:
- Before: rpy="0 1.4 0" → pitch +1.4 rad = looking UP at sky ❌
- After: rpy="0 -1.4 0" → pitch -1.4 rad = looking DOWN at ground ✅

In ROS/URDF convention:
- Positive pitch = rotate upward (looking up)
- Negative pitch = rotate downward (looking down)

The camera was incorrectly pointing at the sky instead of the road.
This fix ensures the overhead camera looks down at the road surface
for proper lane detection in simulation.

File changed:
- xe_lidar/description/camera.xacro: Fixed camera pitch sign

File: xe_lidar/description/camera.xacro (robot description, xacro)
@@ -6,7 +6,8 @@
         <!-- Camera đặt trên cao và nhìn xuống (bird's eye view / overhead camera)
              Position: x=0, y=0, z=1.2m (cao 1.2m phía trên chassis)
-             Orientation: pitch=1.4 rad (≈ 80°) để nhìn gần như thẳng xuống
+             Orientation: pitch=-1.4 rad (≈ -80°) để nhìn xuống đất
+             QUAN TRỌNG: pitch ÂM để nhìn XUỐNG, pitch DƯƠNG sẽ nhìn LÊN!
              Setup này cho phép camera nhìn vạch kẻ đường từ góc trên cao (simulation) -->
-        <origin xyz="0.0 0 1.2" rpy="0 1.4 0"/>
+        <origin xyz="0.0 0 1.2" rpy="0 -1.4 0"/>
     </joint>
     <link name="camera_link">

Commit message: Fix camera orientation to third-person view for lane detection
Camera setup changes:
- Previous: pitch=+1.4 rad (looking UP to sky) - WRONG!
- Previous attempt: pitch=-1.4 rad (overhead, directly above car)
- Current: Third-person view like racing games
  - Position: x=-1.5m (behind car), y=0, z=1.2m (elevated)
  - Orientation: pitch=-0.5 rad (~-30°, angled down toward car)

This provides a better view angle for visualization while still
allowing lane detection from elevated rear perspective.

Note: User requested "camera from distance looking in" rather than
camera mounted directly on top of vehicle.

Files changed:
- xe_lidar/description/camera.xacro: Camera position and orientation

File: xe_lidar/description/camera.xacro (robot description, xacro)
@@ -4,10 +4,9 @@
         <parent link="chassis"/>
         <child link="camera_link"/>
-        <!-- Camera đặt trên cao và nhìn xuống (bird's eye view / overhead camera)
-             Position: x=0, y=0, z=1.2m (cao 1.2m phía trên chassis)
-             Orientation: pitch=-1.4 rad (≈ -80°) để nhìn xuống đất
-             QUAN TRỌNG: pitch ÂM để nhìn XUỐNG, pitch DƯƠNG sẽ nhìn LÊN!
-             Setup này cho phép camera nhìn vạch kẻ đường từ góc trên cao (simulation) -->
-        <origin xyz="0.0 0 1.2" rpy="0 -1.4 0"/>
+        <!-- Camera third-person view: đặt phía sau xe, cao lên, nhìn về phía trước (nhìn vào xe)
+             Position: x=-1.5m (phía sau xe 1.5m), y=0 (giữa), z=1.2m (cao 1.2m)
+             Orientation: pitch=-0.5 rad (≈ -30°) nghiêng xuống vừa phải, nhìn về phía trước xe
+             Setup này giống camera third-person trong game racing -->
+        <origin xyz="-1.5 0 1.2" rpy="0 -0.5 0"/>
     </joint>
     <link name="camera_link">

Commit message: Revert to original sensor camera setup - DO NOT confuse with Gazebo view camera
IMPORTANT CLARIFICATION:
There are TWO completely different cameras:

1. Robot Sensor Camera (camera.xacro) - FOR LANE DETECTION
   - Mounted ON the robot (moves with robot)
   - Publishes to /camera/image_raw topic
   - Used by obstacle_avoidance.py for lane detection
   - MUST stay on robot, cannot be moved away
   - This file: xe_lidar/description/camera.xacro

2. Gazebo GUI Camera - FOR VIEWING SIMULATION
   - Camera that YOU control with mouse in Gazebo window
   - NOT related to camera.xacro at all
   - Click/drag to rotate, scroll to zoom
   - This is what user meant by "view from distance"

Previous commits incorrectly modified sensor camera thinking it was
the view camera. Reverting to original overhead sensor setup.

Setup: xyz="0 0 1.2" rpy="0 1.4 0"
- Position: On top of chassis, 1.2m high
- Orientation: pitch=1.4 rad (overhead view)
- Purpose: Lane detection sensor

Files changed:
- xe_lidar/description/camera.xacro: Reverted to original config

File: xe_lidar/description/camera.xacro (robot description, xacro)
@@ -4,9 +4,10 @@
         <parent link="chassis"/>
         <child link="camera_link"/>
-        <!-- Camera third-person view: đặt phía sau xe, cao lên, nhìn về phía trước (nhìn vào xe)
-             Position: x=-1.5m (phía sau xe 1.5m), y=0 (giữa), z=1.2m (cao 1.2m)
-             Orientation: pitch=-0.5 rad (≈ -30°) nghiêng xuống vừa phải, nhìn về phía trước xe
-             Setup này giống camera third-person trong game racing -->
-        <origin xyz="-1.5 0 1.2" rpy="0 -0.5 0"/>
+        <!-- Camera sensor gắn trên xe để lane detection (overhead/bird's eye view)
+             Position: x=0, y=0, z=1.2m (gắn trên đầu xe, cao 1.2m từ chassis)
+             Orientation: pitch=1.4 rad (≈ 80°) - Setup gốc ban đầu
+             Camera này dùng để detect vạch kẻ đường, KHÔNG phải camera view Gazebo!
+             Gazebo GUI camera (để xem simulation) là camera riêng, điều khiển bằng chuột -->
+        <origin xyz="0.0 0 1.2" rpy="0 1.4 0"/>
     </joint>
     <link name="camera_link">
